File: kicad/ChristmasLEDs/ChristmasLEDs.sch (KiCad schematic (older format))
At the start: 20 parts, among them J1 Power, J2 PIR, J3 Relay, J4 LEDs, J6 Button1, U1 74HC245, U2 ESP32-DevKitC

Commit message: Update board error!!
Connections:
- net GPIO4: no longer J2.3 (Pin_3), R5.2
- net GPIO16: now reaches U2.27 (GPIO16)
- net GPIO16: now also J2.3 (Pin_3), R5.2
Changed lines of the file:
@@
 Wire Wire Line
 	3550 5800 3800 5800
-Text Label 3800 5800 0    50   ~ 0
-GPIO4
 $Comp
 L Connector:Conn_01x02_Male J6
@@
 Wire Wire Line
 	2700 6650 2900 6650
+Wire Wire Line
+	6200 3900 6450 3900
+Text Label 6450 3900 0    50   ~ 0
+GPIO16
+Text Label 3800 5800 0    50   ~ 0
+GPIO16
 $EndSCHEMATC
